File: thermocouples.kicad_pcb (KiCad board)
At the start: 2 copper layers, 24 x 48 mm, 21 parts, among them J1 Conn_02x15_Odd_Even, J2 Conn_02x15_Odd_Even, J3 Conn_01x02, J4 Conn_01x02, U1 ADS1120-RVA

Commit message: sourced all components on lcsc, added ibom and outputs
Parts:
- R7, R8: value R -> 0.47
